File: kicad_board/multieff.kicad_pcb (KiCad board)
At the start: 2 copper layers, 120 x 80 mm, 33 parts, among them J1 Wha1

Commit message: Add missing screen alim connector
Parts:
- added ScrAl1: Conn_01x02, Connector_JST:JST_XH_B2B-XH-AM_1x02_P2.50mm_Vertical, F.Cu at (47.0, 47.2)
- moved C1 7.00 mm to (55.8, 46.5)
- moved C2 6.75 mm to (56.3, 53.2)
Routing:
- net /5V: track 0.00 -> 9.96 mm

Commit message: Improved expression pedal handling
Parts:
- removed J1: Wha1, Connector_JST:JST_XH_B3B-XH-AM_1x03_P2.50mm_Vertical
- added J2: Conn_01x01_Socket, Connector_PinSocket_2.54mm:PinSocket_1x01_P2.54mm_Vertical, F.Cu at (45.5, 58.5)
- added R6: 10k, Resistor_THT:R_Axial_DIN0309_L9.0mm_D3.2mm_P12.70mm_Horizontal, F.Cu at (56.2, 75.5)
- added WhaJack1: Wha1, Connector_JST:JST_XH_B3B-XH-AM_1x03_P2.50mm_Vertical, F.Cu at (49.8, 83.2)
Connections:
- ADC1 pad 6: Net-(ADC1-Pin_6) -> unconnected-(ADC1-Pin_6-Pad6)
- ADC1 pad 9: unconnected-(ADC1-Pin_9-Pad9) -> Net-(ADC1-Pin_9)
- Pisound1 pad 6: unconnected-(Pisound1-Pin_6-Pad6) -> Net-(J2-Pin_1)
Routing:
- net Net-(ADC1-Pin_9): track 0.00 -> 13.4 mm
- net Net-(ADC1-Pin_6): track 13.0 -> 0.00 mm
- net Net-(J2-Pin_1): track 0.00 -> 4.52 mm
